File: USB-C-Breakout HW/Type-C-Breakout.kicad_pcb (KiCad board)
At the start: 2 copper layers, 23 x 19.4 mm, 10 parts, among them J1 USB_C_Receptacle_USB2.0_14P, J2 Conn_01x04_MountingPin

Commit message: More files :)
Parts:
- added G***: LOGO, Logos:Github, F.Cu at (152.8, 49.5)
- added G***: LOGO, Logos:Github, B.Cu at (173.2, 49.5)
Other:
- board text added: "vmshade"

Commit message: dasodfjkl
Parts:
- removed the G*** at (173.2, 49.5)
Changed lines of the file:
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@@
-		(embedded_fonts no)
-	)
-	(footprint "Logos:Github"
-		(layer "B.Cu")
-		(at 173.15 49.45 -90)
-		(property "Reference" "G***"
-			(at 0 0 90)
-			(layer "B.SilkS")
-			(hide yes)
-			(effects
-				(font
-					(size 1.5 1.5)
-					(thickness 0.3)
-				)
-				(justify mirror)
-			)
-		)
-		(property "Value" "LOGO"
-			(at 0.75 0 90)
-			(layer "B.SilkS")
-			(hide yes)
-			(effects
-				(font
-					(size 1.5 1.5)
-					(thickness 0.3)
-				)
-				(justify mirror)
-			)
-		)
-		(property "Datasheet" ""
-			(at 0 0 90)
-			(layer "B.Fab")
-			(hide yes)
-			(effects
-				(font
-					(size 1.27 1.27)
-					(thickness 0.15)
-				)
-				(justify mirror)
-			)
-		)
-		(property "Description" ""
-			(at 0 0 90)
-			(layer "B.Fab")
-			(hide yes)
-			(effects
-				(font
-					(size 1.27 1.27)
-					(thickness 0.15)
-				)
-				(justify mirror)
-			)
-		)
-		(attr board_only exclude_from_pos_files exclude_from_bom)
-		(fp_poly
-			(pts
-				(xy 0.08781 0.45263) (xy 0.145619 0.43696) (xy 0.190587 0.418724) (xy 0.239305 0.392461) (xy 0.282904 0.361418)
-				(xy 0.323797 0.323866) (xy 0.326002 0.321592) (xy 0.367386 0.273311) (xy 0.401014 0.222223) (xy 0.427083 0.167898)
-				(xy 0.445786 0.109907) (xy 0.45732 0.04782) (xy 0.459384 0.028641) (xy 0.460993 -0.033525) (xy 0.45467 -0.094257)
-				(xy 0.440778 -0.152943) (xy 0.419678 -0.208974) (xy 0.391733 -0.261738) (xy 0.357305 -0.310624)
-				(xy 0.316757 -0.355021) (xy 0.270449 -0.39432) (xy 0.218745 -0.427908) (xy 0.176034 -0.449254) (xy 0.156816 -0.457208)
-				(xy 0.143177 -0.461287) (xy 0.133397 -0.461645) (xy 0.125758 -0.458437) (xy 0.120833 -0.454221)
-				(xy 0.117998 -0.450906) (xy 0.115894 -0.446643) (xy 0.114418 -0.440254) (xy 0.113468 -0.430559)
-				(xy 0.112942 -0.416378) (xy 0.112738 -0.396535) (xy 0.11275 -0.369847) (xy 0.112776 -0.361497) (xy 0.112711 -0.32874)
-				(xy 0.112125 -0.30299) (xy 0.110825 -0.282928) (xy 0.108615 -0.267232) (xy 0.105302 -0.254583) (xy 0.100691 -0.24366)
-				(xy 0.094588 -0.233141) (xy 0.093686 -0.231753) (xy 0.08935 -0.224262) (xy 0.090766 -0.220835) (xy 0.098607 -0.218723)
-				(xy 0.132666 -0.21097) (xy 0.16003 -0.203224) (xy 0.182307 -0.1948) (xy 0.201109 -0.18501) (xy 0.218045 -0.173169)
-				(xy 0.23058 -0.162448) (xy 0.254936 -0.134719) (xy 0.27319 -0.101574) (xy 0.285389 -0.062889) (xy 0.29158 -0.018538)
-				(xy 0.292413 0.002824) (xy 0.290967 0.038649) (xy 0.285357 0.069065) (xy 0.275043 0.096168) (xy 0.263048 0.116862)
-				(xy 0.254246 0.131315) (xy 0.250272 0.141578) (xy 0.250376 0.14965) (xy 0.250521 0.150201) (xy 0.252686 0.163927)
-				(xy 0.253581 0.182896) (xy 0.253267 0.204121) (xy 0.251801 0.224616) (xy 0.249242 0.241395) (xy 0.24867 0.24379)
-				(xy 0.244745 0.256489) (xy 0.240436 0.263071) (xy 0.234193 0.265669) (xy 0.232618 0.265894) (xy 0.21978 0.264946)
-				(xy 0.202068 0.26033) (xy 0.181651 0.252835) (xy 0.160695 0.243251) (xy 0.142621 0.23315) (xy 0.116462 0.216864)
-				(xy 0.08636 0.223629) (xy 0.062727 0.227382) (xy 0.033579 0.229661) (xy 0.001602 0.230467) (xy -0.030515 0.229801)
-				(xy -0.060085 0.227661) (xy -0.084421 0.22405) (xy -0.086479 0.223604) (xy -0.116699 0.216815) (xy -0.138571 0.230576)
-				(xy -0.165985 0.245906) (xy -0.19301 0.257504) (xy -0.217208 0.264359) (xy -0.221958 0.265137) (xy -0.233464 0.266207)
-				(xy -0.23982 0.264472) (xy -0.244059 0.258717) (xy -0.245523 0.255698) (xy -0.248798 0.244298) (xy -0.251336 0.227275)
-				(xy -0.252996 0.207296) (xy -0.253641 0.187026) (xy -0.253129 0.169132) (xy -0.251319 0.15628) (xy -0.250827 0.154656)
-				(xy -0.24881 0.146619) (xy -0.249771 0.139325) (xy -0.254483 0.130041) (xy -0.260377 0.120976) (xy -0.27536 0.095891)
-				(xy -0.285198 0.071747) (xy -0.290685 0.045775) (xy -0.292615 0.015206) (xy -0.292643 0.008335)
-				(xy -0.290192 -0.036211) (xy -0.28293 -0.074753) (xy -0.270507 -0.108325) (xy -0.252575 -0.137963)
-				(xy -0.237087 -0.156363) (xy -0.218711 -0.173224) (xy -0.197719 -0.187158) (xy -0.172756 -0.198773)
-				(xy -0.142466 -0.208676) (xy -0.105494 -0.217476) (xy -0.09664 -0.219261) (xy -0.087012 -0.221154)
-				(xy -0.096129 -0.235907) (xy -0.103474 -0.250117) (xy -0.109644 -0.265809) (xy -0.11034 -0.268061)
-				(xy -0.116548 -0.280975) (xy -0.127013 -0.289445) (xy -0.142974 -0.294097) (xy -0.164611 -0.295554)
-				(xy -0.191235 -0.291814) (xy -0.214741 -0.280435) (xy -0.233762 -0.262567) (xy -0.254171 -0.238204)
-				(xy -0.271327 -0.220203) (xy -0.286272 -0.207779) (xy -0.300044 -0.200149) (xy -0.313682 -0.196529)
-				(xy -0.32206 -0.195957) (xy -0.332905 -0.197679) (xy -0.336313 -0.203086) (xy -0.332283 -0.212194)
-				(xy -0.320808 -0.225018) (xy -0.314192 -0.23114) (xy -0.298913 -0.246205) (xy -0.286999 -0.261958)
-				(xy -0.276033 -0.281721) (xy -0.273415 -0.287131) (xy -0.256647 -0.316316) (xy -0.237269 -0.33788)
-				(xy -0.214434 -0.352311) (xy -0.187292 -0.360099) (xy -0.155001 -0.361731) (xy -0.144982 -0.361156)
-				(xy -0.112519 -0.358653) (xy -0.112519 -0.402279) (xy -0.112707 -0.422407) (xy -0.113463 -0.435991)
-				(xy -0.115074 -0.44482) (xy -0.117824 -0.450678) (xy -0.120854 -0.454241) (xy -0.127635 -0.459695)
-				(xy -0.135084 -0.461824) (xy -0.145085 -0.460505) (xy -0.159522 -0.455616) (xy -0.170916 -0.450994)
-				(xy -0.22743 -0.423174) (xy -0.278316 -0.38923) (xy -0.323775 -0.348995) (xy -0.364007 -0.302305)
-				(xy -0.382954 -0.275379) (xy -0.413811 -0.221032) (xy -0.437018 -0.164107) (xy -0.452588 -0.105312)
-				(xy -0.460532 -0.045351) (xy -0.460858 0.015067) (xy -0.453581 0.075234) (xy -0.43871 0.134445)
-				(xy -0.416256 0.191992) (xy -0.38623 0.247168) (xy -0.37454 0.264912) (xy -0.357831 0.28654) (xy -0.336279 0.310635)
-				(xy -0.312015 0.335096) (xy -0.287165 0.35782) (xy -0.263859 0.376708) (xy -0.25472 0.383207) (xy -0.201869 0.413939)
-				(xy -0.146331 0.437086) (xy -0.088849 0.452588) (xy -0.030169 0.460386) (xy 0.028966 0.46042)
-			)
-			(stroke
-				(width 0)
-				(type solid)
-			)
-			(fill yes)
-			(layer "B.SilkS")
-		)
 		(embedded_fonts no)
 	)
@@
 		)
 	)
-	(gr_text "vmshade"
-		(at 173.600001 50 90)
-		(layer "B.SilkS")
-		(effects
-			(font
-				(size 1 1)
-				(thickness 0.25)
-				(bold yes)
-			)
-			(justify left bottom mirror)
-		)
-	)
